File: Keybord.kicad_pcb (KiCad board)
At the start: 2 copper layers, 236 parts, among them IC1 74AHCT1G125DBVRG4, J1 USB_C_Receptacle_USB2.0_14P, SW1 SW_Push, SW10 SW_Push, SW11 SW_Push, SW12 SW_Push, SW13 SW_Push, SW14 SW_Push, SW15 SW_Push, SW16 SW_Push, SW17 SW_Push, SW18 SW_Push, SW19 SW_Push, SW2 SW_Push, SW20 SW_Push, SW21 SW_Push, SW22 SW_Push, SW23 SW_Push, SW24 SW_Push, SW25 SW_Push, SW26 SW_Push, SW27 SW_Push, SW28 SW_Push, SW29 SW_Push, SW3 SW_Push, SW30 SW_Push, SW31 SW_Push, SW32 SW_Push, SW33 SW_Push, SW34 SW_Push, SW35 SW_Push, SW36 SW_Push, SW37 SW_Push, SW38 SW_Push, SW39 SW_Push, SW4 SW_Push, SW40 SW_Push, SW41 SW_Push, SW42 SW_Push, SW43 SW_Push, SW44 SW_Push, SW45 SW_Push, SW46 SW_Push, SW47 SW_Push, SW48 SW_Push, SW49 SW_Push, SW5 SW_Push, SW50 SW_Push, SW51 SW_Push, SW52 SW_Push, SW53 SW_Push, SW54 SW_Push, SW55 SW_Push, SW56 SW_Push, SW57 SW_Push, SW58 SW_Push, SW59 SW_Push, SW6 SW_Push, SW60 SW_Push, SW61 SW_Push, SW62 SW_Push, SW63 SW_Push, SW64 SW_Push, SW65 SW_Push, SW66 SW_Push, SW67 SW_Push, SW68 SW_Push, SW69 SW_Push, SW7 SW_Push, SW70 SW_Push, SW71 SW_Push, SW72 SW_Push, SW73 SW_Push, SW74 SW_Push, SW75 SW_Push, SW76 SW_Push, SW77 SW_Push, SW78 SW_Push, SW8 SW_Push, SW9 SW_Push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

Commit message: Switch Layout on PCB
Parts:
- removed the SW56 at (97.6, 155.0)
- D1: value D -> 1N4148
- D10: renamed from D55; value D -> 1N4148
- D11: renamed from D60; value D -> 1N4148
- D12: renamed from D65; value D -> 1N4148
- D13: renamed from D70; value D -> 1N4148
- D14: renamed from D74; value D -> 1N4148
- D15: renamed from D2; value D -> 1N4148
- D16: renamed from D8; value D -> 1N4148
- D17: renamed from D14; value D -> 1N4148
- D18: renamed from D20; value D -> 1N4148
- D19: renamed from D26; value D -> 1N4148
- D2: renamed from D7; value D -> 1N4148
- D20: renamed from D32; value D -> 1N4148
- D21: renamed from D38; value D -> 1N4148
- D22: renamed from D44; value D -> 1N4148
- D23: renamed from D50; value D -> 1N4148
- D24: renamed from D56; value D -> 1N4148
- D25: renamed from D61; value D -> 1N4148
- D26: renamed from D66; value D -> 1N4148
- D27: renamed from D71; value D -> 1N4148
- D28: renamed from D75; value D -> 1N4148
- D29: renamed from D3; value D -> 1N4148
- D3: renamed from D13; value D -> 1N4148
- D30: renamed from D9; value D -> 1N4148
- D31: renamed from D15; value D -> 1N4148
- D32: renamed from D21; value D -> 1N4148
- D33: renamed from D27; value D -> 1N4148
- D34: renamed from D33; value D -> 1N4148
- D35: renamed from D39; value D -> 1N4148
- D36: renamed from D45; value D -> 1N4148
- D37: renamed from D51; value D -> 1N4148
- D38: renamed from D57; value D -> 1N4148
- D39: renamed from D62; value D -> 1N4148
- D4: renamed from D19; value D -> 1N4148
- D40: renamed from D67; value D -> 1N4148
- D41: renamed from D72; value D -> 1N4148
- D42: renamed from D76; value D -> 1N4148
- D43: renamed from D4; value D -> 1N4148
- D44: renamed from D10; value D -> 1N4148
- D45: renamed from D16; value D -> 1N4148
- D46: renamed from D22; value D -> 1N4148
- D47: renamed from D28; value D -> 1N4148
- D48: renamed from D34; value D -> 1N4148
- D49: renamed from D40; value D -> 1N4148
- D5: renamed from D25; value D -> 1N4148
- D50: renamed from D46; value D -> 1N4148
- D51: renamed from D52; value D -> 1N4148
- D52: renamed from D58; value D -> 1N4148
- D53: renamed from D63; value D -> 1N4148
- D54: renamed from D68; value D -> 1N4148
- D55: renamed from D73; value D -> 1N4148
- D56: renamed from D5; value D -> 1N4148
- D57: renamed from D11; value D -> 1N4148
- D58: renamed from D17; value D -> 1N4148
- D59: renamed from D23; value D -> 1N4148
- D6: renamed from D31; value D -> 1N4148
- D60: renamed from D29; value D -> 1N4148
- D61: renamed from D35; value D -> 1N4148
- D62: renamed from D41; value D -> 1N4148
- D63: renamed from D47; value D -> 1N4148
- D64: renamed from D53; value D -> 1N4148
- D65: renamed from D59; value D -> 1N4148
- D66: renamed from D64; value D -> 1N4148
- D67: renamed from D69; value D -> 1N4148
- D68: renamed from D6; value D -> 1N4148
- D69: renamed from D12; value D -> 1N4148
- D7: renamed from D37; value D -> 1N4148
- D70: renamed from D18; value D -> 1N4148
- D71: renamed from D24; value D -> 1N4148
- D72: renamed from D30; value D -> 1N4148
- D73: renamed from D36; value D -> 1N4148
- D74: renamed from D42; value D -> 1N4148
- D75: renamed from D48; value D -> 1N4148
- D76: renamed from D54; value D -> 1N4148
- D8: renamed from D43; value D -> 1N4148
- D9: renamed from D49; value D -> 1N4148
- moved SW79 268.9 mm to (409.5, 234.5)
- moved SW78 256.5 mm to (391.5, 233.0)
- moved C13 225.8 mm to (394.4, 209.7)
- moved C14 225.8 mm to (394.4, 212.7)
- moved C2 225.8 mm to (394.4, 206.7)
- moved C3 225.8 mm to (427.4, 134.9)
- moved D10 225.8 mm to (358.4, 141.3)
- moved D104 225.8 mm to (397.4, 136.2)
- moved D105 225.8 mm to (397.4, 142.9)
- moved D106 225.8 mm to (397.4, 149.5)
- moved D107 225.8 mm to (397.4, 156.1)
- moved D108 225.8 mm to (397.4, 162.7)
- moved D109 225.8 mm to (397.4, 169.3)
- moved D11 225.8 mm to (358.4, 158.1)
- moved D110 225.8 mm to (397.4, 176.0)
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- renumbered SW57 to SW10, SW62 to SW11, SW67 to SW12, SW72 to SW13, SW76 to SW14, SW4 to SW15, SW10 to SW16, SW16 to SW17, SW22 to SW18, SW28 to SW19, SW9 to SW2, SW34 to SW20, SW40 to SW21, SW46 to SW22, SW52 to SW23, SW58 to SW24, SW63 to SW25, SW68 to SW26, SW73 to SW27, SW77 to SW28, SW5 to SW29, SW15 to SW3, SW11 to SW30, SW17 to SW31, SW23 to SW32, SW29 to SW33, SW35 to SW34, SW41 to SW35, SW47 to SW36, SW53 to SW37, SW59 to SW38, SW64 to SW39, SW21 to SW4, SW69 to SW40, SW74 to SW41, SW78 to SW42, SW6 to SW43, SW12 to SW44, SW18 to SW45, SW24 to SW46, SW30 to SW47, SW36 to SW48, SW42 to SW49, SW27 to SW5, SW48 to SW50, SW54 to SW51, SW60 to SW52, SW65 to SW53, SW70 to SW54, SW75 to SW55, SW7 to SW56, SW13 to SW57, SW19 to SW58, SW25 to SW59, SW33 to SW6, SW31 to SW60, SW37 to SW61, SW43 to SW62, SW49 to SW63, SW55 to SW64, SW61 to SW65, SW71 to SW67, SW8 to SW68, SW14 to SW69, SW39 to SW7, SW20 to SW70, SW26 to SW71, SW32 to SW72, SW38 to SW73, SW44 to SW74, SW50 to SW75, SW2 to SW78, SW3 to SW79, SW45 to SW8, SW51 to SW9

Commit message: Fix routing on Shematic, PCB Diode Place, ROW routing
Parts:
- removed D76: 1N4148, Diode_SMD:D_SOD-123
- moved D14 348.3 mm to (33.0, 53.5), turned to 90 degrees
- moved D28 339.4 mm to (37.5, 72.5), turned to 90 degrees
- moved D42 333.1 mm to (40.0, 91.5), turned to 90 degrees
- moved D55 332.1 mm to (35.5, 110.5), turned to 90 degrees
- moved D68 300.4 mm to (35.5, 129.8), turned to 90 degrees
- moved D3 292.0 mm to (84.5, 25.0), turned to 90 degrees
- moved D16 284.1 mm to (71.0, 53.5), turned to 90 degrees
- moved D29 282.2 mm to (61.5, 72.3), turned to 90 degrees
- moved D56 280.7 mm to (57.0, 110.3), turned to 90 degrees
- moved D69 279.3 mm to (59.0, 130.0), turned to 90 degrees
- moved D43 273.9 mm to (66.5, 91.5), turned to 90 degrees
- moved D30 269.7 mm to (80.5, 72.5), turned to 90 degrees
- moved D4 269.1 mm to (103.5, 24.9), turned to 90 degrees
- moved D57 265.5 mm to (76.0, 110.5), turned to 90 degrees
- moved D17 263.7 mm to (90.0, 53.5), turned to 90 degrees
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Connections:
- SW72 pad 1: COL4 -> COL9
- SW73 pad 1: COL5 -> COL10
- SW74 pad 1: COL6 -> COL11
- SW75 pad 1: COL7 -> COL12
Routing:
- net COL3: track 0.00 -> 152.2 mm
- net COL0: track 0.00 -> 135.3 mm
- net COL1: track 0.00 -> 128.4 mm
- net COL2: track 0.00 -> 126.4 mm
- net COL11: track 0.00 -> 125.8 mm
- net COL9: track 0.00 -> 125.7 mm
- net COL10: track 0.00 -> 123.5 mm
- net COL12: track 0.00 -> 113.5 mm
- net COL6: track 0.00 -> 102.6 mm
- net COL7: track 0.00 -> 101.0 mm
- net COL5: track 0.00 -> 100.1 mm
- net COL4: track 0.00 -> 99.4 mm
- net COL8: track 0.00 -> 98.1 mm
- net Net-(D73-A): track 0.00 -> 3.71 mm
- net Net-(D72-A): track 0.00 -> 3.63 mm
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